File: tsl2585-breakout.kicad_sch (KiCad schematic)
At the start: 0 parts

Commit message: Schematic for breakout board complete
Parts:
- added C2: 1uF, Capacitor_SMD:C_0402_1005Metric, symbol Device:C_Small
- added C4: 4.7uF, Capacitor_SMD:C_0402_1005Metric, symbol Device:C_Small
- added C9 (x2): 1uF, Capacitor_SMD:C_0603_1608Metric, symbol Device:C_Small
- added J1: Conn_01x08, Connector_PinHeader_2.54mm:PinHeader_1x08_P2.54mm_Vertical, symbol Connector_Generic:Conn_01x08
- added R1: 22R, Resistor_SMD:R_0402_1005Metric, symbol Device:R_Small
- added R4 (x3): 10K, Resistor_SMD:R_0603_1608Metric, symbol Device:R_Small
- added U1: TSL2585, lib_fp:AMS_TSL2585_OLGA-6_2x1mm_P0.65mm, symbol AMS_Sensor_Optical:TSL2585
- added U2: MIC5365-1.8YC5, Package_TO_SOT_SMD:SOT-353_SC-70-5, symbol Regulator_Linear:MIC5365-3.3YC5
Connections:
- new net: C2.1, R1.1, U1.1 (VDD)
- new net +1V8: C4.1, C9.2, J1.2 (Pin_2), R1.2, U2.5 (VOUT)
- new net GND: C2.2, C4.2, C9.1, C9.1, J1.8 (Pin_8), U1.3 (VSS), U2.2 (GND)
- new net SENSOR_INT: J1.6 (Pin_6), R4.2, U1.5 (INT)
- new net SENSOR_SCL: J1.4 (Pin_4), R4.2, U1.4 (SCL)
- new net SENSOR_SDA: J1.5 (Pin_5), R4.2, U1.6 (SDA)
- new net SENSOR_VSYNC: J1.7 (Pin_7), U1.2 (VSYNC/GPIO)
- new net VCC: C9.2, J1.1 (Pin_1), U2.1 (VIN), U2.3 (EN)
- new net V_{PU}: J1.3 (Pin_3), R4.1, R4.1, R4.1
Other:
- note added: "Connector and Pullups"
- note added: "Light sensor"
- note added: "Power supply"
