File: tsl2585-breakout.kicad_sch (KiCad schematic)
At the start: 11 parts, among them J1 Conn_01x08, U1 TSL2585, U2 MIC5365-1.8YC5

Commit message: PCB layout done
Parts:
- added H1, H2: MountingHole, MountingHole:MountingHole_2.5mm_Pad, symbol Mechanical:MountingHole
Changed lines of the file:
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@@
+    )
+  )
+  (symbol (lib_id "Mechanical:MountingHole") (at 23.495 85.725 0) (unit 1)
+    (in_bom yes) (on_board yes) (dnp no) (fields_autoplaced)
+    (property "Reference" "H2" (at 26.67 84.455 0)
+      (effects (font (size 1.27 1.27)) (justify left))
+    )
+    (property "Value" "MountingHole" (at 26.67 86.995 0)
+      (effects (font (size 1.27 1.27)) (justify left))
+    )
+    (property "Footprint" "MountingHole:MountingHole_2.5mm_Pad" (at 23.495 85.725 0)
+      (effects (font (size 1.27 1.27)) hide)
+    )
+    (property "Datasheet" "~" (at 23.495 85.725 0)
+      (effects (font (size 1.27 1.27)) hide)
+    )
+    (property "Description" "" (at 23.495 85.725 0)
+      (effects (font (size 1.27 1.27)) hide)
+    )
+    (property "Manufacturer" "" (at 23.495 85.725 0)
+      (effects (font (size 1.27 1.27)) hide)
+    )
+    (property "Manufacturer PN" "" (at 23.495 85.725 0)
+      (effects (font (size 1.27 1.27)) hide)
+    )
+    (property "Supplier" "" (at 23.495 85.725 0)
+      (effects (font (size 1.27 1.27)) hide)
+    )
+    (property "Supplier PN" "" (at 23.495 85.725 0)
+      (effects (font (size 1.27 1.27)) hide)
+    )
+    (instances
+      (project "tsl2585-breakout"
+        (path "/3f3ab8a6-b03e-4a96-9558-b31e20a6d8cc"
+          (reference "H2") (unit 1)
+        )
+      )
     )
   )
@@
         )
       )
+    )
+  )
+  (symbol (lib_id "Mechanical:MountingHole") (at 23.495 80.01 0) (unit 1)
+    (in_bom yes) (on_board yes) (dnp no) (fields_autoplaced)
+    (property "Reference" "H1" (at 26.67 78.74 0)
+      (effects (font (size 1.27 1.27)) (justify left))
+    )
+    (property "Value" "MountingHole" (at 26.67 81.28 0)
+      (effects (font (size 1.27 1.27)) (justify left))
+    )
+    (property "Footprint" "MountingHole:MountingHole_2.5mm_Pad" (at 23.495 80.01 0)
+      (effects (font (size 1.27 1.27)) hide)
+    )
+    (property "Datasheet" "~" (at 23.495 80.01 0)
+      (effects (font (size 1.27 1.27)) hide)
+    )
+    (property "Description" "" (at 23.495 80.01 0)
+      (effects (font (size 1.27 1.27)) hide)
+    )
+    (property "Manufacturer" "" (at 23.495 80.01 0)
+      (effects (font (size 1.27 1.27)) hide)
+    )
+    (property "Manufacturer PN" "" (at 23.495 80.01 0)
+      (effects (font (size 1.27 1.27)) hide)
+    )
+    (property "Supplier" "" (at 23.495 80.01 0)
+      (effects (font (size 1.27 1.27)) hide)
+    )
+    (property "Supplier PN" "" (at 23.495 80.01 0)
+      (effects (font (size 1.27 1.27)) hide)
+    )
+    (instances
+      (project "tsl2585-breakout"
+        (path "/3f3ab8a6-b03e-4a96-9558-b31e20a6d8cc"
+          (reference "H1") (unit 1)
+        )
+      )
