File: tsl2585-breakout.kicad_pcb (KiCad board)
At the start: 2 copper layers, 0 parts

Commit message: PCB layout done
Parts:
- added C1: 1uF, Capacitor_SMD:C_0402_1005Metric, F.Cu at (40.8, 28.0)
- added C2: 4.7uF, Capacitor_SMD:C_0402_1005Metric, F.Cu at (40.2, 29.5)
- added C3: 1uF, Capacitor_SMD:C_0603_1608Metric, F.Cu at (35.0, 30.9)
- added C4: 1uF, Capacitor_SMD:C_0603_1608Metric, F.Cu at (35.0, 35.8)
- added H1: MountingHole, MountingHole:MountingHole_2.5mm_Pad, F.Cu at (33.0, 26.0)
- added H2: MountingHole, MountingHole:MountingHole_2.5mm_Pad, F.Cu at (52.0, 26.0)
- added J1: Conn_01x08, Connector_PinHeader_2.54mm:PinHeader_1x08_P2.54mm_Vertical, F.Cu at (33.6, 39.0)
- added R1: 22R, Resistor_SMD:R_0402_1005Metric, F.Cu at (39.7, 28.0)
- added R2: 10K, Resistor_SMD:R_0603_1608Metric, F.Cu at (41.2, 35.3)
- added R3: 10K, Resistor_SMD:R_0603_1608Metric, F.Cu at (43.8, 35.3)
- added R4: 10K, Resistor_SMD:R_0603_1608Metric, F.Cu at (46.3, 35.3)
- added U1: TSL2585, lib_fp:AMS_TSL2585_OLGA-6_2x1mm_P0.65mm, F.Cu at (42.5, 28.0)
- added U2: MIC5365-1.8YC5, Package_TO_SOT_SMD:SOT-353_SC-70-5, F.Cu at (35.0, 33.4)
Routing:
- net +1V8: track 0.00 -> 26.3 mm
- net /SENSOR_VSYNC: track 0.00 -> 20.3 mm, vias 0 -> 2
- net /SENSOR_INT: track 0.00 -> 15.6 mm, vias 0 -> 2
- net /V_{PU}: track 0.00 -> 15.6 mm, vias 0 -> 3
- net /SENSOR_SDA: track 0.00 -> 14.4 mm
- net /SENSOR_SCL: track 0.00 -> 11.5 mm
- net VCC: track 0.00 -> 7.68 mm
- net GND: track 0.00 -> 7.61 mm, vias 0 -> 3
- net Net-(U1-VDD): track 0.00 -> 2.58 mm
- added copper zone on B.Cu, net GND
Other:
- board outline added: 25 x 18.5 mm
